File: hardware/FRC-ButtonBoard/carrierboard.sch (EAGLE design)
At the start: 36 parts

Commit message: commit to more buttons
Parts:
- removed JGPIO_1_2, JGPIO_3_4: (no value), pinhead:PINHD-2X3
- added C3: 0.1uF, SparkFun-Capacitors:0.1UF-KIT-EZ-50V-20%
- added J1: USB_A_SMT_FEMALE, SparkFun-Connectors:USB_A_SMT_FEMALE
- added JBTN25, JBTN26, JBTN27, JBTN28: (no value), SparkFun-Connectors:CONN_06SILK_FEMALE_PTH
- added JRST: (no value), pinhead:PINHD-1X2
- added JUSB: USB_B_PTH, SparkFun-Connectors:USB_B_PTH
- added P1: J1B1211CCD, WIZnet:J1B1211CCD
Connections:
- removed net GPIO1: JGPIO_1_2.5, U$1.38-A14/CS/IN1
- removed net GPIO2: JGPIO_1_2.6, U$1.39-A15/CS/OUT1A
- removed net GPIO3: JGPIO_3_4.5, U$1.40-A16/CS1
- removed net GPIO4: JGPIO_3_4.6, U$1.41-A17/MISO1
- new net B25_DIN: JBTN24.6, JBTN25.5
- new net B26_DIN: JBTN25.6, JBTN26.5
- new net B27_DIN: JBTN26.6, JBTN27.5
- new net B28_DIN: JBTN27.6, JBTN28.5
- new net BTN25: JBTN25.1, U$1.38-A14/CS/IN1
- new net BTN26: JBTN26.1, U$1.39-A15/CS/OUT1A
- new net BTN27: JBTN27.1, U$1.40-A16/CS1
- new net BTN28: JBTN28.1, U$1.41-A17/MISO1
- new net ETH_LED: P1.GRN+, U$1.LED
- new net ETH_R+: P1.RD+, U$1.R+
- new net ETH_R-: P1.RD-, U$1.R-
- new net ETH_T+: P1.TD+, U$1.T+
- new net ETH_T-: P1.TD-, U$1.T-
- new net N$1: C3.2, P1.RCT, P1.TCT
- new net N$10: U$1.VUSB
- new net PROGRAM_RESET: JRST.1, U$1.PROGRAM
- new net USBH_D+: J1.D+, U$1.DP
- new net USBH_D-: J1.D-, U$1.DM
- new net USB_D+: JUSB.D+, U$1.D+
- new net USB_D-: JUSB.D-, U$1.D-
- net 3V3: no longer JGPIO_1_2.1, JGPIO_1_2.2, JGPIO_3_4.1, JGPIO_3_4.2
- net 5V: now also J1.VBUS, JBTN25.3, JBTN26.3, JBTN27.3, JBTN28.3, JUSB.VBUS, U$1.5V
- net B_DOUT: now also JBTN28.6; no longer JBTN24.6
- net GND: now also C3.1, J1.GND, J1.SHIELD, JBTN25.2, JBTN25.4, JBTN26.2, JBTN26.4, JBTN27.2, JBTN27.4, JBTN28.2, JBTN28.4, JRST.2, JUSB.GND, JUSB.SHIELD, P1.CH_GND@2, P1.CH_GND@3, P1.GH_GND@1, P1.GRN-, U$1.G; no longer JGPIO_1_2.3, JGPIO_1_2.4, JGPIO_3_4.3, JGPIO_3_4.4
Other:
- moved on the sheet: C1, C2
